File: arthurc.sch (KiCad schematic (older format))
At the start: 59 parts, among them IC1 ATMEGA328, P1 I/O, P10 CD2, P11 CD2, P12 CD1, P13 CD1, P4 CONN_6, P5 CONN_6, P6 9VBAT, P7 GPS_UP501, P8 FTDI, P9 ISP, SW1 SW_PUSH, U1 3V3, U2 74HC125, U3 5V0, X1 CRYSTAL_2

Commit message: ArthurC work in progress
Parts:
- removed B1, B12, B13, B14, B7, B9: I/O, I/O, symbol I/O
- removed P7: GPS_UP501, PIN_ARRAY-6X1, symbol CONN_6
- removed X1: CRYSTAL_2, Xtal_SMD2, symbol CRYSTAL_2
- added X1: 16MHz, symbol CRYSTAL
- P7: renamed from P?; value CONN_9 -> GPS
Connections:
- net labels removed: +5V, ADC6, GPS_3V3, PC0, VIN
- wire segments 232 -> 227
- no-connect marks 15 -> 13
Other:
- note added: "VIN"
- note removed: "PD2 (1pps)\nGPS 1pps signal"
- note removed: "PD7 (SQW)\nRTC 1Hz signal"
- moved on the sheet: C7, D1, D2, D3, D4, P1, P10, P11, P12, P13, P4, P5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
