File: KiCAD/arthurc.kicad_pcb (KiCad board)
At the start: 2 copper layers, 63.5 x 30.5 mm, 63 parts, among them IC1 ATMEGA328, P1 I/O, P10 CD2, P11 CD2, P12 CD1, P13 CD1, P14 I/O, P15 I/O, P16 I/O, P4 CONN_6, P5 CONN_6, P6 9VBAT, P7 GPS, P8 FTDI, P9 ISP, SW1 SW_PUSH, U1 3V3, U2 74HC125, U3 5V0, U4 DS3231N, X1 16MHz

Commit message: board layout work in progress
Parts:
- removed C3: 2u2 Tant, ArthurC Lib:c_0805
- removed C4: 100n, ArthurC Lib:c_0805
- removed C6: 47u,10V, ArthurC Lib:C_ELCO_SMD
- removed C8: 100n, ArthurC Lib:d_0805
- removed G1, G2: Logo-WL3, Logo-WL3
- removed G3: LOGO, OSHW_6mm
- removed R3, R4, R6: 10k, ArthurC Lib:r_0805
- removed U2: 74HC125, ArthurC Lib:SO14E
- removed U3: 5V0, ArthurC Lib:SOT23-5
- added B1: AREF, ArthurC Lib:I%2fO, F.Cu at (54.2, 49.8)
- added P2: BAT, ArthurC Lib:pin_strip_2, F.Cu at (81.6, 32.0)
- BT1: value BATT_RTC -> Batt_RTC
- C10, C11, C7, C9: footprint ArthurC Lib:d_0805 -> ArthurC Lib:c_0805
- P6: value 9VBAT -> LiPo
- R5, R8: value 1k5 -> 750E
- SD1: value SD_CARD_MICRO -> SD_CARD_Micro
- X1: value 16MHz -> 8MHz
- moved B8 2.54 mm to (56.7, 49.8)
Connections:
- B19 pad 1: /arthurc_rtc/5V0 -> +3.3V
- C1 pad 1: /arthurc_rtc/5V0 -> +3.3V
- C2 pad 1: /arthurc_rtc/5V0 -> /arthurc_rtc/BAT
- IC1 pad 18: /arthurc_rtc/5V0 -> +3.3V
- IC1 pad 20: /arthurc_rtc/5V0 -> Net-(B1-Pad1)
- IC1 pad 4: /arthurc_rtc/5V0 -> +3.3V
- IC1 pad 6: /arthurc_rtc/5V0 -> +3.3V
- P1 pad 1: Net-(P1-Pad1) -> (no net)
- P10 pad 3: /arthurc_rtc/5V0 -> +3.3V
- P11 pad 3: /arthurc_rtc/5V0 -> +3.3V
- P14 pad 1: +3.3V -> /3Vgps
- P4 pad 3: /arthurc_rtc/5V0 -> (no net)
- P4 pad 6: Net-(P4-Pad6) -> (no net)
- P5 pad 1: Net-(P5-Pad1) -> (no net)
- P5 pad 2: Net-(P5-Pad2) -> (no net)
- P5 pad 3: Net-(P5-Pad3) -> (no net)
- P5 pad 4: Net-(P5-Pad4) -> (no net)
- P6 pad 1: /+9V -> /arthurc_rtc/BAT
- P7 pad 1: +3.3V -> /3Vgps
- P7 pad 8: /arthurc_rtc/5V0 -> +3.3V
- P8 pad 3: /arthurc_rtc/5V0 -> +3.3V
- P9 pad 2: /arthurc_rtc/5V0 -> +3.3V
- R1 pad 1: /arthurc_rtc/5V0 -> +3.3V
- R2 pad 1: /arthurc_rtc/5V0 -> +3.3V
- R7 pad 1: /arthurc_rtc/5V0 -> +3.3V
- R9 pad 1: /arthurc_rtc/5V0 -> +3.3V
- SD1 pad 1: Net-(SD1-Pad1) -> (no net)
- SD1 pad 2: /SD_CS -> /SS
- SD1 pad 3: /SD_DATA_IN -> /MOSI
- SD1 pad 5: /SD_CLK -> /SCK
- SD1 pad 8: Net-(SD1-Pad8) -> (no net)
- SD1 pad 9: Net-(SD1-Pad9) -> (no net)
- SD1 pad H1: Net-(SD1-PadH1) -> (no net)
- SD1 pad H2: Net-(SD1-PadH2) -> (no net)
- U1 pad 3: /arthurc_rtc/5V0 -> /arthurc_rtc/BAT
- U4 pad 2: /arthurc_rtc/5V0 -> +3.3V
Routing:
- net /arthurc_rtc/5V0: track 254.6 -> 0.00 mm, vias 6 -> 0
- net +3.3V: track 141.7 -> 314.9 mm, vias 6 -> 11
- net /arthurc_rtc/BAT: track 87.0 -> 117.2 mm
- net /SD_CS: track 19.3 -> 0.00 mm, vias 2 -> 0
- net GND: track 359.5 -> 340.7 mm
- net /SS: track 34.4 -> 52.7 mm, vias 2 -> 4
- net /SCK: track 65.8 -> 48.1 mm, vias 3 -> 4
- net /+9V: track 16.1 -> 0.00 mm
- net /MOSI: track 47.7 -> 40.4 mm, vias 3 -> 1
- net Net-(B1-Pad1): track 0.00 -> 5.50 mm
- net /SD_DATA_IN: track 4.92 -> 0.00 mm
- net /SD_CLK: track 4.89 -> 0.00 mm
- net /GPS_Rx: track 65.6 -> 69.3 mm
- net /GPS_Tx: track 71.6 -> 74.2 mm
- net Net-(C4-Pad1): track 2.65 -> 0.00 mm
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