File: KiCAD/arthurc.sch (KiCad schematic (older format))
At the start: 46 parts, among them IC1 ATMEGA328, P1 I/O, P10 CD2, P11 CD2, P12 CD1, P13 CD1, P14 I/O, P15 I/O, P16 I/O, P2 BAT, P4 CONN_6, P5 CONN_6, P6 LiPo, P7 GPS, P8 FTDI, P9 ISP, SW1 SW_PUSH, U1 3V3, X1 8MHz

Commit message: Board layout work in progress
Parts:
- added C3: 47uF_25V, ArthurC Lib:C_ELCO_SMD, symbol C_POL
- B1: footprint (none) -> ArthurC Lib:I%2fO
- C1, C10, C11, C2, C5, C7: footprint c_0805 -> ArthurC Lib:c_0805
- D1, D2: footprint d_0805 -> ArthurC Lib:d_0805
- IC1: footprint TQFP32 -> ArthurC Lib:TQFP32
- P10, P11, P12, P13: footprint Sck-04-F-SMT -> ArthurC Lib:Sck-04-F-SMT
- P2: footprint (none) -> ArthurC Lib:pin_strip_2
- P4, P5, P8: footprint PIN_ARRAY-6X1 -> ArthurC Lib:PIN_ARRAY-6X1
- P6: footprint pin_strip_2 -> ArthurC Lib:pin_strip_2
- P9: footprint ISP -> ArthurC Lib:ISP
- PCB1: footprint PCB -> ArthurC Lib:PCB
- R1, R2, R5, R7, R8: footprint r_0805 -> ArthurC Lib:r_0805
- SC1: footprint vite_3mm -> ArthurC Lib:vite_3mm
- SD1: footprint (none) -> ArthurC Lib:SD_Micro
- SW1: footprint SW_SMD -> ArthurC Lib:SW_SMD
- U1: footprint SOT23-3 -> ArthurC Lib:SOT23-3
Connections:
- net BAT: now also C3.1
- net GND: now also C3.2
Changed lines of the file:
@@
 	5150 4900 6050 4900
 Wire Wire Line
-	9325 2400 10600 2400
+	9325 2400 10925 2400
 Wire Wire Line
 	6050 4900 6050 4750
@@
 F 0 "C11" H 725 3225 50  0000 L CNN
 F 1 "22p" H 725 3425 50  0000 L CNN
-F 2 "c_0805" H 700 3325 60  0001 C CNN
+F 2 "ArthurC Lib:c_0805" H 700 3325 60  0001 C CNN
 F 3 "" H 700 3325 60  0001 C CNN
 F 4 "490-1734-1-ND" H 700 3525 60  0001 C CNN "Digikey"
@@
 F 0 "C10" H 725 2875 50  0000 L CNN
 F 1 "22p" H 725 2675 50  0000 L CNN
-F 2 "c_0805" H 700 2775 60  0001 C CNN
+F 2 "ArthurC Lib:c_0805" H 700 2775 60  0001 C CNN
 F 3 "" H 700 2775 60  0001 C CNN
 F 4 "490-1734-1-ND" H 700 2975 60  0001 C CNN "Digikey"
@@
 F 0 "PCB1" H 10800 5875 60  0000 C CNN
 F 1 "PCB" H 10800 6475 60  0000 C CNN
-F 2 "PCB" H 10800 6175 60  0001 C CNN
+F 2 "ArthurC Lib:PCB" H 10800 6175 60  0001 C CNN
 F 3 "" H 10800 6175 60  0001 C CNN
 	1    10800 6175
@@
 F 0 "P5" V 4925 7375 60  0000 C CNN
 F 1 "CONN_6" V 5025 7375 60  0000 C CNN
-F 2 "PIN_ARRAY-6X1" H 4975 7375 60  0001 C CNN
+F 2 "ArthurC Lib:PIN_ARRAY-6X1" H 4975 7375 60  0001 C CNN
 F 3 "" H 4975 7375 60  0001 C CNN
 	1    4975 7375
@@
 F 0 "P4" V 4925 6650 60  0000 C CNN
 F 1 "CONN_6" V 5025 6650 60  0000 C CNN
-F 2 "PIN_ARRAY-6X1" H 4975 6650 60  0001 C CNN
+F 2 "ArthurC Lib:PIN_ARRAY-6X1" H 4975 6650 60  0001 C CNN
 F 3 "" H 4975 6650 60  0001 C CNN
 	1    4975 6650
@@
 F 0 "P6" V 10775 700 40  0000 C CNN
 F 1 "LiPo" V 10875 700 40  0000 C CNN
-F 2 "pin_strip_2" H 10825 700 60  0001 C CNN
+F 2 "ArthurC Lib:pin_strip_2" H 10825 700 60  0001 C CNN
 F 3 "" H 10825 700 60  0001 C CNN
 	1    10825 700
@@
 F 0 "C5" H 9375 2200 50  0000 L CNN
 F 1 "1u" H 9375 2000 50  0000 L CNN
-F 2 "c_0805" H 9325 2100 60  0001 C CNN
+F 2 "ArthurC Lib:c_0805" H 9325 2100 60  0001 C CNN
 F 3 "" H 9325 2100 60  0001 C CNN
 	1    9325 2100
@@
 F 0 "P12" V 8325 6200 50  0000 C CNN
 F 1 "CD1" V 8425 6200 50  0000 C CNN
-F 2 "Sck-04-F-SMT" H 8375 6200 60  0001 C CNN
+F 2 "ArthurC Lib:Sck-04-F-SMT" H 8375 6200 60  0001 C CNN
 F 3 "" H 8375 6200 60  0001 C CNN
 	1    8375 6200
@@
 F 0 "P11" V 8325 5750 50  0000 C CNN
 F 1 "CD2" V 8425 5750 50  0000 C CNN
-F 2 "Sck-04-F-SMT" H 8375 5750 60  0001 C CNN
+F 2 "ArthurC Lib:Sck-04-F-SMT" H 8375 5750 60  0001 C CNN
 F 3 "" H 8375 5750 60  0001 C CNN
 	1    8375 5750
@@
 F 0 "P13" V 7500 6200 50  0000 C CNN
 F 1 "CD1" V 7600 6200 50  0000 C CNN
-F 2 "Sck-04-F-SMT" H 7550 6200 60  0001 C CNN
+F 2 "ArthurC Lib:Sck-04-F-SMT" H 7550 6200 60  0001 C CNN
 F 3 "" H 7550 6200 60  0001 C CNN
 	1    7550 6200
@@
 F 0 "P10" V 7500 5750 50  0000 C CNN
 F 1 "CD2" V 7600 5750 50  0000 C CNN
-F 2 "Sck-04-F-SMT" H 7550 5750 60  0001 C CNN
+F 2 "ArthurC Lib:Sck-04-F-SMT" H 7550 5750 60  0001 C CNN
 F 3 "" H 7550 5750 60  0001 C CNN
 	1    7550 5750
@@
 F 0 "R8" V 3855 6750 50  0000 C CNN
 F 1 "750E" V 3775 6750 50  0000 C CNN
-F 2 "r_0805" H 3775 6750 60  0001 C CNN
+F 2 "ArthurC Lib:r_0805" H 3775 6750 60  0001 C CNN
 F 3 "" H 3775 6750 60  0001 C CNN
 	1    3775 6750
@@
 F 0 "R5" V 3555 6750 50  0000 C CNN
 F 1 "750E" V 3475 6750 50  0000 C CNN
-F 2 "r_0805" H 3475 6750 60  0001 C CNN
+F 2 "ArthurC Lib:r_0805" H 3475 6750 60  0001 C CNN
 F 3 "" H 3475 6750 60  0001 C CNN
 	1    3475 6750
@@
 F 0 "D2" H 3775 7350 50  0000 C CNN
 F 1 "LED" H 3775 7150 50  0000 C CNN
-F 2 "d_0805" H 3775 7250 60  0001 C CNN
+F 2 "ArthurC Lib:d_0805" H 3775 7250 60  0001 C CNN
 F 3 "" H 3775 7250 60  0001 C CNN
 	1    3775 7250
@@
 F 0 "D1" H 3475 7350 50  0000 C CNN
 F 1 "LED" H 3475 7150 50  0000 C CNN
-F 2 "d_0805" H 3475 7250 60  0001 C CNN
+F 2 "ArthurC Lib:d_0805" H 3475 7250 60  0001 C CNN
 F 3 "" H 3475 7250 60  0001 C CNN
 	1    3475 7250
@@
 F 0 "P9" V 1200 7050 60  0000 C CNN
 F 1 "ISP" V 1300 7050 60  0000 C CNN
-F 2 "ISP" H 1250 7050 60  0001 C CNN
+F 2 "ArthurC Lib:ISP" H 1250 7050 60  0001 C CNN
 F 3 "" H 1250 7050 60  0001 C CNN
 	1    1250 7050
@@
 F 0 "SC1" H 10800 5500 40  0000 C CNN
 F 1 "SCREW" H 10800 5700 40  0001 C CNN
-F 2 "vite_3mm" H 10800 5600 60  0001 C CNN
+F 2 "ArthurC Lib:vite_3mm" H 10800 5600 60  0001 C CNN
 F 3 "" H 10800 5600 60  0001 C CNN
 	1    10800 5600
@@
 F 0 "C7" V 2100 6750 50  0000 L CNN
 F 1 "100n" V 2025 6750 50  0000 L CNN
-F 2 "c_0805" H 2250 6750 60  0001 C CNN
+F 2 "ArthurC Lib:c_0805" H 2250 6750 60  0001 C CNN
 F 3 "" H 2250 6750 60  0001 C CNN
 	1    2250 6750
@@
 F 0 "P8" V 2850 7050 60  0000 C CNN
 F 1 "FTDI" V 2950 7050 60  0000 C CNN
-F 2 "PIN_ARRAY-6X1" H 2900 7050 60  0001 C CNN
+F 2 "ArthurC Lib:PIN_ARRAY-6X1" H 2900 7050 60  0001 C CNN
 F 3 "" H 2900 7050 60  0001 C CNN
 	1    2900 7050
@@
 F 0 "U1" H 9800 1800 60  0000 C CNN
 F 1 "3V3" H 10100 1800 60  0000 C CNN
-F 2 "SOT23-3" H 9950 1950 60  0001 C CNN
+F 2 "ArthurC Lib:SOT23-3" H 9950 1950 60  0001 C CNN
 F 3 "" H 9950 1950 60  0001 C CNN
 F 4 "MCP1700T-3302E/TT" H 9950 1950 60  0001 C CNN "Part No"
@@
 F 0 "R2" V 5080 1450 50  0000 C CNN
 F 1 "10k" V 5000 1450 50  0000 C CNN
-F 2 "r_0805" H 5000 1450 60  0001 C CNN
+F 2 "ArthurC Lib:r_0805" H 5000 1450 60  0001 C CNN
 F 3 "" H 5000 1450 60  0001 C CNN
 	1    5000 1450
@@
 F 0 "R1" V 4875 1450 50  0000 C CNN
 F 1 "10k" V 4800 1450 50  0000 C CNN
-F 2 "r_0805" H 4800 1450 60  0001 C CNN
+F 2 "ArthurC Lib:r_0805" H 4800 1450 60  0001 C CNN
 F 3 "" H 4800 1450 60  0001 C CNN
 	1    4800 1450
@@
 F 0 "SW1" H 1225 4460 50  0000 C CNN
 F 1 "SW_PUSH" H 1075 4270 50  0000 C CNN
-F 2 "SW_SMD" H 1075 4350 60  0001 C CNN
+F 2 "ArthurC Lib:SW_SMD" H 1075 4350 60  0001 C CNN
 F 3 "" H 1075 4350 60  0001 C CNN
 F 4 "" H 1325 4560 60  0001 C CNN "DigiKey"
@@
 F 0 "R7" H 1125 1900 50  0000 C CNN
 F 1 "10k" V 1075 1700 50  0000 C CNN
-F 2 "r_0805" H 1075 1700 60  0001 C CNN
+F 2 "ArthurC Lib:r_0805" H 1075 1700 60  0001 C CNN
 F 3 "" H 1075 1700 60  0001 C CNN
 	1    1075 1700
@@
 F 0 "C1" H 1300 1325 50  0000 L CNN
 F 1 "100n" H 1300 1125 50  0000 L CNN
-F 2 "c_0805" H 1250 1225 60  0001 C CNN
+F 2 "ArthurC Lib:c_0805" H 1250 1225 60  0001 C CNN
 F 3 "" H 1250 1225 60  0001 C CNN
 	1    1250 1225
@@
 F 0 "C2" H 10650 2200 50  0000 L CNN
 F 1 "1u" H 10650 2000 50  0000 L CNN
-F 2 "c_0805" H 10600 2100 60  0001 C CNN
+F 2 "ArthurC Lib:c_0805" H 10600 2100 60  0001 C CNN
 F 3 "" H 10600 2100 60  0001 C CNN
 	1    10600 2100
@@
 F 0 "IC1" H 1700 4400 50  0000 L BNN
 F 1 "ATMEGA328" H 1750 2500 50  0000 L BNN
-F 2 "TQFP32" H 2925 1675 50  0001 C CNN
+F 2 "ArthurC Lib:TQFP32" H 2925 1675 50  0001 C CNN
 F 3 "" H 2400 3250 60  0001 C CNN
 	1    2400 3250
@@
 F 0 "SD1" H 5475 5000 50  0000 C CNN
 F 1 "SD_CARD_Micro" H 5675 5075 50  0000 C CNN
-F 2 "" H 5300 4550 60  0000 C CNN
+F 2 "ArthurC Lib:SD_Micro" H 5300 4550 60  0001 C CNN
 F 3 "" H 5300 4550 60  0000 C CNN
 	1    5300 4550
@@
 F 0 "B1" V 2025 1375 50  0000 L CNN
 F 1 "AREF" V 1925 1400 50  0000 C CNN
-F 2 "" H 1850 1400 60  0000 C CNN
+F 2 "ArthurC Lib:I%2fO" H 1850 1400 60  0001 C CNN
 F 3 "" H 1850 1400 60  0000 C CNN
 	1    1850 1400
@@
 F 0 "P2" V 9050 700 40  0000 C CNN
 F 1 "BAT" V 9150 700 40  0000 C CNN
-F 2 "" H 9100 700 60  0000 C CNN
+F 2 "ArthurC Lib:pin_strip_2" H 9100 700 60  0001 C CNN
 F 3 "" H 9100 700 60  0000 C CNN
 	1    9100 700
@@
 Connection ~ 9900 1100
 Wire Wire Line
-	10925 1850 10925 1050
+	10925 1050 10925 1900
+$Comp
+L C_POL C3
+U 1 1 536B66B9
+P 10925 2100
+F 0 "C3" H 10825 2200 50  0000 L CNN
+F 1 "47uF_25V" H 10925 1950 50  0000 L CNN
+F 2 "ArthurC Lib:C_ELCO_SMD" H 10925 2100 60  0001 C CNN
+F 3 "" H 10925 2100 60  0000 C CNN
+	1    10925 2100
+	1    0    0    -1
+$EndComp
+Connection ~ 10925 1850
+Wire Wire Line
+	10925 2400 10925 2350
+Connection ~ 10600 2400
 $EndSCHEMATC
