File: KiCAD/arthurc_rtc.sch (KiCad schematic (older format))
At the start: 7 parts, among them U4 DS3231N

Commit message: Ultimate GPS header added to I2GPS
Parts:
- B15, B2, B3: footprint I/O -> ArthurC Lib:I%2fO
Changed lines of the file:
@@
 $EndComp
 $Comp
-L +BATT #PWR010
+L +BATT #PWR8
 U 1 1 4EC101F0
 P 5300 1850
-F 0 "#PWR010" H 5300 1800 20  0001 C CNN
+F 0 "#PWR8" H 5300 1800 20  0001 C CNN
 F 1 "+BATT" H 5300 1950 30  0000 C CNN
 F 2 "" H 5300 1850 60  0001 C CNN
@@
 F 0 "B15" H 6905 2750 40  0000 L CNN
 F 1 "I/O" H 6825 2805 30  0001 C CNN
-F 2 "I/O" H 6825 2750 60  0001 C CNN
+F 2 "ArthurC Lib:I%2fO" H 6825 2750 60  0001 C CNN
 F 3 "" H 6825 2750 60  0001 C CNN
 	1    6825 2750
@@
 F 0 "B3" H 6905 2600 40  0000 L CNN
 F 1 "I/O" H 6825 2655 30  0001 C CNN
-F 2 "I/O" H 6825 2600 60  0001 C CNN
+F 2 "ArthurC Lib:I%2fO" H 6825 2600 60  0001 C CNN
 F 3 "" H 6825 2600 60  0001 C CNN
 	1    6825 2600
@@
 F 0 "B2" H 6905 2450 40  0000 L CNN
 F 1 "I/O" H 6825 2505 30  0001 C CNN
-F 2 "I/O" H 6825 2450 60  0001 C CNN
+F 2 "ArthurC Lib:I%2fO" H 6825 2450 60  0001 C CNN
 F 3 "" H 6825 2450 60  0001 C CNN
 	1    6825 2450

Commit message: work in progress, converting design to work on 3V3
Parts:
- removed BT1: BATT_RTC, CR1632, symbol BATT_RTC
- added BT1: Batt_RTC, symbol Batt_RTC
Connections:
- net labels added: 3V3
- net labels removed: 5V0
Changed lines of the file:
@@
 $EndComp
 $Comp
-L +BATT #PWR8
+L +BATT #PWR08
 U 1 1 4EC101F0
 P 5300 1850
-F 0 "#PWR8" H 5300 1800 20  0001 C CNN
+F 0 "#PWR08" H 5300 1800 20  0001 C CNN
 F 1 "+BATT" H 5300 1950 30  0000 C CNN
 F 2 "" H 5300 1850 60  0001 C CNN
@@
 SCL
 Text HLabel 7250 3750 2    60   Input ~ 0
-5V0
+3V3
 Text Label 7050 3750 0    40   ~ 0
-5V0
+3V3
 Text Label 7050 4125 0    40   ~ 0
 GND
@@
 U 1 1 4E1FEA7E
 P 4175 2775
-F 0 "C9" V 4225 2875 50  0000 L CNN
-F 1 "100n" V 4225 2575 50  0000 L CNN
+F 0 "C9" H 4200 2675 50  0000 L CNN
+F 1 "100n" H 4150 2375 50  0000 L CNN
 F 2 "c_0805" H 4175 2775 60  0001 C CNN
 F 3 "" H 4175 2775 60  0001 C CNN
@@
 32k
 $Comp
-L BATT_RTC BT1
-U 1 1 4E1FEA78
+L Batt_RTC BT1
+U 1 1 535D65B7
 P 3950 2800
-F 0 "BT1" H 3650 2600 50  0000 C CNN
-F 1 "BATT_RTC" H 3950 2610 50  0000 C CNN
-F 2 "CR1632" H 3950 2800 60  0001 C CNN
-F 3 "" H 3950 2800 60  0001 C CNN
-F 4 "BU2032SM-HD-GCT-ND " H 3950 2800 60  0001 C CNN "Digikey"
+F 0 "BT1" V 3875 2575 50  0000 C CNN
+F 1 "Batt_RTC" V 3950 2500 50  0000 C CNN
+F 2 "" H 3950 2800 60  0000 C CNN
+F 3 "" H 3950 2800 60  0000 C CNN
+F 4 "BU2032SM-HD-GCT-ND " H 4050 3100 60  0001 C CNN "Digikey"
 	1    3950 2800
 	0    1    1    0

Commit message: Board layout work in progress
Parts:
- BT1: footprint (none) -> ArthurC Lib:CR1632
- C9: footprint c_0805 -> ArthurC Lib:c_0805
- R9: footprint r_0805 -> ArthurC Lib:r_0805
- U4: footprint DS3231 -> ArthurC Lib:DS3231
Changed lines of the file:
@@
 F 0 "R9" V 6730 2000 50  0000 C CNN
 F 1 "10k" V 6650 2000 50  0000 C CNN
-F 2 "r_0805" H 6650 2000 60  0001 C CNN
+F 2 "ArthurC Lib:r_0805" H 6650 2000 60  0001 C CNN
 F 3 "" H 6650 2000 60  0001 C CNN
 	1    6650 2000
@@
 F 0 "U4" H 5850 3350 60  0000 C CNN
 F 1 "DS3231N" H 5250 2400 60  0000 C CNN
-F 2 "DS3231" H 5550 2800 60  0001 C CNN
+F 2 "ArthurC Lib:DS3231" H 5550 2800 60  0001 C CNN
 F 3 "" H 5550 2800 60  0001 C CNN
 	1    5550 2800
@@
 F 0 "C9" H 4200 2675 50  0000 L CNN
 F 1 "100n" H 4150 2375 50  0000 L CNN
-F 2 "c_0805" H 4175 2775 60  0001 C CNN
+F 2 "ArthurC Lib:c_0805" H 4175 2775 60  0001 C CNN
 F 3 "" H 4175 2775 60  0001 C CNN
 	1    4175 2775
@@
 F 0 "BT1" V 3875 2575 50  0000 C CNN
 F 1 "Batt_RTC" V 3950 2500 50  0000 C CNN
-F 2 "" H 3950 2800 60  0000 C CNN
+F 2 "ArthurC Lib:CR1632" H 3950 2800 60  0001 C CNN
 F 3 "" H 3950 2800 60  0000 C CNN
 F 4 "BU2032SM-HD-GCT-ND " H 4050 3100 60  0001 C CNN "Digikey"
