File: KiCAD/rev2/arthurc.sch (KiCad schematic (older format))
At the start: 47 parts, among them IC1 ATMEGA328, P1 I/O, P10 CD2, P11 CD2, P12 CD1, P13 CD1, P14 I/O, P15 I/O, P16 I/O, P2 BAT, P4 CONN_6, P5 CONN_6, P6 LiPo, P7 GPS, P8 FTDI, P9 ISP, SW1 SW_PUSH, U1 3V3, X1 8MHz

Commit message: ArthurC rev2 work in progress
Parts:
- removed B1: AREF, ArthurC Lib:I%2fO, symbol I/O
- added CON?: USB-MINI-B, symbol USB-MINI-B
- added U?: ATMEGA32U4-A, TQFP44, symbol ATMEGA32U4-A
- SW1: value SW_PUSH -> RST
Connections:
- net +3.3V: now also U?.14 (VCC), U?.24 (AVCC), U?.34 (VCC), U?.44 (AVCC); no longer IC1.18 (AVCC)
- net GND: now also C11.2; no longer C11.1
- net RESET: now also U?.13 (~RESET~); no longer IC1.29 (PC6(/RESET))
- net PB6 renamed XTAL1
- net XTAL1: now also U?.17 (XTAL1); no longer IC1.7 (PB6(XTAL1/TOSC1))
- removed net PB7: C11.2, IC1.8 (PB7(XTAL2/TOSC2)), X1.2
- new net XTAL2: C11.1, U?.16 (XTAL2), X1.2
Other:
- moved on the sheet: C10, C11, R7, SW1, X1

Commit message: ArthurC rev2 work in progress
Parts:
- added R? (x2): 22E, symbol R
Connections:
- net GND: now also CON?.5 (GND), CON?.6 (SHELL1), CON?.7 (SHELL2), CON?.8 (SHELL3), CON?.9 (SHELL4)
- net 5V0: now reaches CON?.1 (VBUS)
- net USBD-: now reaches CON?.2 (D-)
- net USBD-: now also R?.2
- net USBD+: now reaches CON?.3 (D+)
- net USBD+: now also R?.2
- new net D+: R?.1
- new net D-: R?.1
- no-connect marks 13 -> 14
Other:
- moved on the sheet: CON?
Changed lines of the file:
@@
 	4375 4150 4500 4150
 Wire Wire Line
-	-3200 2550 -3125 2550
-Wire Wire Line
-	-3125 2550 -2875 2550
+	-3200 2550 -2875 2550
 Connection ~ 4525 6700
 Wire Wire Line
@@
 	3400 3550 3625 3550
 Wire Wire Line
-	5750 800  5750 1100
-Wire Wire Line
 	5300 4400 4750 4400
 Wire Wire Line
@@
 Wire Wire Line
 	4750 4400 4750 4550
-Connection ~ 7600 1100
-Wire Wire Line
-	1250 1425 1250 2450
-Wire Wire Line
-	1250 2450 1250 4975
+Wire Wire Line
+	1250 1425 1250 4975
 Wire Wire Line
 	4650 4350 3400 4350
 Connection ~ 5950 4900
 Wire Wire Line
-	2350 4850 2350 4975
-Wire Wire Line
-	2350 4975 2350 5100
+	2350 4850 2350 5100
 Connection ~ 2450 4975
 Wire Wire Line
@@
 Connection ~ 1250 800
 Wire Wire Line
-	9950 2350 9950 2400
-Wire Wire Line
-	9950 2400 9950 2475
+	9950 2350 9950 2475
 Wire Wire Line
 	4650 4300 4650 4350
@@
 	3775 7500 3775 7450
 Wire Wire Line
-	3475 7500 3625 7500
-Wire Wire Line
-	3625 7500 3775 7500
+	3475 7500 3775 7500
 Wire Wire Line
 	3475 7500 3475 7450
@@
 	2550 7100 1650 7100
 Wire Wire Line
-	5750 1100 7600 1100
-Wire Wire Line
 	7600 1100 9000 1100
 Wire Wire Line
-	9000 1050 9000 1100
-Wire Wire Line
-	9000 1100 9000 1850
-Wire Wire Line
-	9000 1850 9325 1850
-Wire Wire Line
-	9325 1850 9400 1850
-Wire Wire Line
-	10500 1850 10600 1850
-Wire Wire Line
-	10600 1850 10925 1850
-Wire Wire Line
-	1075 800  1250 800
-Wire Wire Line
-	1250 800  2350 800
-Wire Wire Line
-	2350 800  2450 800
-Wire Wire Line
-	2450 800  4425 800
-Wire Wire Line
-	4425 800  4800 800
-Wire Wire Line
-	4800 800  5000 800
-Wire Wire Line
-	5000 800  5750 800
-Wire Wire Line
-	1650 7300 2350 7300
-Wire Wire Line
-	2350 7300 2550 7300
+	9000 1050 9000 1850
+Wire Wire Line
+	9000 1850 9400 1850
+Wire Wire Line
+	10500 1850 10925 1850
+Wire Wire Line
+	1075 800  5000 800
+Wire Wire Line
+	1650 7300 2550 7300
 Wire Wire Line
 	2550 6900 1650 6900
@@
 	4625 6400 4225 6400
 Wire Wire Line
-	4225 6700 4525 6700
-Wire Wire Line
-	4525 6700 4625 6700
+	4225 6700 4625 6700
 Wire Notes Line
 	3100 6300 1500 6300
@@
 	4625 7625 4225 7625
 Wire Wire Line
-	-3200 3050 -3125 3050
-Wire Wire Line
-	-3125 3050 -2875 3050
+	-3200 3050 -2875 3050
 Wire Wire Line
 	4375 4050 4500 4050
 Wire Wire Line
-	4500 4050 4500 4150
-Wire Wire Line
-	4500 4150 4500 4600
+	4500 4050 4500 4600
 Wire Notes Line
 	4425 4600 3325 4600
@@
 	5150 4450 5150 4900
 Wire Wire Line
-	5150 4900 5900 4900
-Wire Wire Line
-	5900 4900 5950 4900
-Wire Wire Line
-	5950 4900 6000 4900
-Wire Wire Line
-	6000 4900 6050 4900
-Wire Wire Line
-	9325 2400 9950 2400
-Wire Wire Line
-	9950 2400 10600 2400
-Wire Wire Line
-	10600 2400 10925 2400
+	5150 4900 6050 4900
+Wire Wire Line
+	9325 2400 10925 2400
 Wire Wire Line
 	6050 4900 6050 4750
@@
 Connection ~ -3125 2550
 Wire Wire Line
-	1250 4975 2350 4975
-Wire Wire Line
-	2350 4975 2450 4975
+	1250 4975 2450 4975
 Wire Wire Line
 	4000 2100 4000 2550
@@
 	9900 5850 10000 5850
 Wire Wire Line
-	2450 4850 2450 4975
-Wire Wire Line
-	2450 4975 2450 5100
+	2450 4850 2450 5100
 $Comp
 L GND #PWR01
@@
 	1    0    0    -1
 $EndComp
-Connection ~ 5000 800
 NoConn ~ 4625 6600
 Text Label 6075 6825 0    40   ~ 0
@@
 3V3
 Wire Wire Line
-	9200 1100 9900 1100
-Wire Wire Line
-	9900 1100 10725 1100
+	9200 1100 10725 1100
 Wire Wire Line
 	10725 1100 10725 1050
@@
 Connection ~ 9900 1100
 Wire Wire Line
-	10925 1050 10925 1850
-Wire Wire Line
-	10925 1850 10925 1900
+	10925 1050 10925 1900
 $Comp
 L C_POL C3
@@
 	-2875 2900 -2875 3050
 Wire Wire Line
-	-3675 2300 -3675 2550
-Wire Wire Line
-	-3675 2550 -3675 2800
-Wire Wire Line
-	-3675 2800 -3675 3050
-Wire Wire Line
-	-3675 3050 -3675 3250
+	-3675 2300 -3675 3250
 $Comp
 L GND #PWR?
@@
 Connection ~ -3675 2550
 Wire Wire Line
-	-2700 2300 -2600 2300
-Wire Wire Line
-	-2600 2300 -2500 2300
+	-2700 2300 -2500 2300
 Wire Wire Line
 	-2600 1825 -2600 2300
@@
 	-1550 2050 -1550 1950
 Wire Wire Line
-	-1550 1950 -1450 1950
-Wire Wire Line
-	-1450 1950 -1200 1950
-Wire Wire Line
-	-1200 1950 -1100 1950
+	-1550 1950 -1100 1950
 Wire Wire Line
 	-1100 1950 -1100 2050
@@
 L USB-MINI-B CON?
 U 1 1 538233D1
-P 425 -575
-F 0 "CON?" H 175 -125 60  0000 C CNN
-F 1 "USB-MINI-B" H 375 -1075 60  0000 C CNN
-F 2 "" H 425 -575 60  0000 C CNN
-F 3 "" H 425 -575 60  0000 C CNN
-	1    425  -575
+P 6550 2900
+F 0 "CON?" H 6300 3350 60  0000 C CNN
+F 1 "USB-MINI-B" H 6500 2400 60  0000 C CNN
+F 2 "" H 6550 2900 60  0000 C CNN
+F 3 "" H 6550 2900 60  0000 C CNN
+	1    6550 2900
 	-1   0    0    1
 $EndComp
+Text Label 4550 800  0    60   ~ 0
+3V3
+$Comp
+L GND #PWR?
+U 1 1 5388A365
+P 7225 3500
+F 0 "#PWR?" H 7225 3500 30  0001 C CNN
+F 1 "GND" H 7225 3430 30  0001 C CNN
+F 2 "" H 7225 3500 60  0001 C CNN
+F 3 "" H 7225 3500 60  0001 C CNN
+	1    7225 3500
+	1    0    0    -1
+$EndComp
+Wire Wire Line
+	7100 2600 7225 2600
+Wire Wire Line
+	7225 2600 7225 3500
+NoConn ~ 7100 2750
+Wire Wire Line
+	7100 2900 7650 2900
+Wire Wire Line
+	7100 3050 7650 3050
+Wire Wire Line
+	7100 3200 7450 3200
+Text Label 7450 2900 0    50   ~ 0
+USBD+
+Text Label 7450 3050 0    50   ~ 0
+USBD-
+Text Label 7450 3200 0    50   ~ 0
+5V0
+Wire Wire Line
+	6000 2600 5900 2600
+Wire Wire Line
+	5900 2600 5900 3425
+Wire Wire Line
+	5900 3425 7225 3425
+Connection ~ 7225 3425
+Wire Wire Line
+	6000 2750 5900 2750
+Connection ~ 5900 2750
+Wire Wire Line
+	6000 3050 5900 3050
+Connection ~ 5900 3050
+Wire Wire Line
+	6000 3200 5900 3200
+Connection ~ 5900 3200
+$Comp
+L R R?
+U 1 1 5388AD88
+P 7900 2900
+F 0 "R?" V 7980 2900 50  0000 C CNN
+F 1 "22E" V 7900 2900 50  0000 C CNN
+F 2 "" H 7900 2900 60  0000 C CNN
+F 3 "" H 7900 2900 60  0000 C CNN
+	1    7900 2900
+	0    1    1    0
+$EndComp
+$Comp
+L R R?
+U 1 1 5388AD9A
+P 7900 3050
+F 0 "R?" V 7980 3050 50  0000 C CNN
+F 1 "22E" V 7900 3050 50  0000 C CNN
+F 2 "" H 7900 3050 60  0000 C CNN
+F 3 "" H 7900 3050 60  0000 C CNN
+	1    7900 3050
+	0    1    1    0
+$EndComp
+Wire Wire Line
+	8150 2900 8375 2900
+Wire Wire Line
+	8150 3050 8375 3050
+Text Label 8375 2900 0    50   ~ 0
+D+
+Text Label 8375 3050 0    50   ~ 0
+D-
 $EndSCHEMATC

Commit message: ArthurC rev2 work in progress
Parts:
- removed C7: 100n, ArthurC Lib:c_0805, symbol C
- removed P6: LiPo, ArthurC Lib:pin_strip_2, symbol CONN_2
- removed P8: FTDI, ArthurC Lib:PIN_ARRAY-6X1, symbol CONN_6
- added C?: 10uF_25V, ArthurC Lib:C_ELCO_SMD, symbol C_POL2
- added D?: DIODE_LED, symbol DIODE_LED
- added R?: R, symbol R2
- added SD?: SD_CARD_Micro, ArthurC Lib:SD_Micro, symbol SD_CARD_Micro
- added SL?: S_LINK_3, symbol S_LINK_3
- C2: symbol C -> C_NPOL
- C3: symbol C_POL -> C_POL2
- C5: value 1u -> 0.1u; symbol C -> C_NPOL
- R? (x2): symbol R -> R2
Connections:
- net 5V0: now also SL?.2
- net BAT: no longer C2.1, C3.1, U1.3 (VIN)
- net GND: now also C?.2, D?.2 (K), SD?.6 (GND), SD?.G1, SD?.G2, SD?.G3, SD?.G4
- net GPS_Rx: now also U?.21 ((TXD/INT3)PD3)
- net GPS_Tx: now also U?.20 ((RXD/INT2)PD2)
- net MISO: now also SD?.5 (CLK)
- net MOSI: now also SD?.3 (DI/CMD)
- net SCK: now also SD?.7 (DO/DAT0)
- net SCL: now also U?.18 ((OC0B/SCL/INT0)PD0)
- net SDA: now also U?.19 ((SDA/INT1)PD1)
- net SS: now also SD?.2 (CS/DAT3)
- net +3.3V renamed 3V3
- net 3V3: now also SD?.4 (VCC); no longer C5.1, P2.1 (P1), U1.2 (VOUT)
- new net: C2.1, C5.1, C?.1, R?.1, U1.2 (VOUT)
- new net: C3.1, SL?.3, U1.3 (VIN)
- new net: P2.1 (P1), SL?.1
- new net: D?.1 (A), R?.2
- no-connect marks 14 -> 20
Other:
- note removed: "External Battery\n3V Max."
- note removed: "External Battery\n9V Max."
- note removed: "FTDI Header"
- note removed: "MCP1700T-3302E/TT"
- moved on the sheet: C10, C11, C3, CON?, P2, R7, R?, SW1, U1, U?, X1
